Commit message: Working finger set

File: urdf/dexhand.xacro (robot description, xacro)
@@ -106,6 +106,6 @@
 <link name="middle-bulk_1">
   <inertial>
-    <origin xyz="0.010646950026404922 -0.0158135798135519 0.030689623412746947" rpy="0 0 0"/>
-    <mass value="0.2319963124821001"/>
+    <origin xyz="0.01064695002640492 -0.0158135798135519 0.030689623412746947" rpy="0 0 0"/>
+    <mass value="0.23199631248210004"/>
     <inertia ixx="0.000258" iyy="0.000268" izz="7.1e-05" ixy="-1.4e-05" iyz="4.2e-05" ixz="4e-05"/>
   </inertial>
@@ -121,24 +121,4 @@
     <geometry>
       <mesh filename="package://dexhand_description/meshes/middle-bulk_1.stl" scale="0.001 0.001 0.001"/>
-    </geometry>
-  </collision>
-</link>
-<link name="pinky-bulk_1">
-  <inertial>
-    <origin xyz="0.014707146884874737 -0.009496610763999918 -0.1955891121635459" rpy="0 0 0"/>
-    <mass value="0.11417768838788588"/>
-    <inertia ixx="0.000111" iyy="0.000112" izz="1e-05" ixy="1e-06" iyz="1.3e-05" ixz="-1e-05"/>
-  </inertial>
-  <visual>
-    <origin xyz="0.02396 0.0224 -0.487266" rpy="0 0 0"/>
-    <geometry>
-      <mesh filename="package://dexhand_description/meshes/pinky-bulk_1.stl" scale="0.001 0.001 0.001"/>
-    </geometry>
-    <material name="silver"/>
-  </visual>
-  <collision>
-    <origin xyz="0.02396 0.0224 -0.487266" rpy="0 0 0"/>
-    <geometry>
-      <mesh filename="package://dexhand_description/meshes/pinky-bulk_1.stl" scale="0.001 0.001 0.001"/>
     </geometry>
   </collision>
@@ -226,10 +206,10 @@
 <link name="pinky-knuckle_1">
   <inertial>
-    <origin xyz="0.006818820473941571 0.0011824337110899058 0.0010801856787571174" rpy="0 0 0"/>
+    <origin xyz="0.006818820473942549 0.0011824337110899266 0.0010801856787569508" rpy="0 0 0"/>
     <mass value="0.016772407452453803"/>
     <inertia ixx="1e-06" iyy="1e-06" izz="1e-06" ixy="-0.0" iyz="-0.0" ixz="-0.0"/>
   </inertial>
   <visual>
-    <origin xyz="0.013416 0.039945 -0.334029" rpy="0 0 0"/>
+    <origin xyz="0.013416 0.038945 -0.334029" rpy="0 0 0"/>
     <geometry>
       <mesh filename="package://dexhand_description/meshes/pinky-knuckle_1.stl" scale="0.001 0.001 0.001"/>
@@ -238,7 +218,267 @@
   </visual>
   <collision>
-    <origin xyz="0.013416 0.039945 -0.334029" rpy="0 0 0"/>
+    <origin xyz="0.013416 0.038945 -0.334029" rpy="0 0 0"/>
     <geometry>
       <mesh filename="package://dexhand_description/meshes/pinky-knuckle_1.stl" scale="0.001 0.001 0.001"/>
+    </geometry>
+  </collision>
+</link>
+<link name="index-plp_1">
+  <inertial>
+    <origin xyz="-0.006869198158126709 -0.006033909809302199 0.022940465298997237" rpy="0 0 0"/>
+    <mass value="0.051567105457974535"/>
+    <inertia ixx="1.1e-05" iyy="1.1e-05" izz="2e-06" ixy="-0.0" iyz="-1e-06" ixz="0.0"/>
+  </inertial>
+  <visual>
+    <origin xyz="0.007269 -0.037678 -0.343728" rpy="0 0 0"/>
+    <geometry>
+      <mesh filename="package://dexhand_description/meshes/index-plp_1.stl" scale="0.001 0.001 0.001"/>
+    </geometry>
+    <material name="silver"/>
+  </visual>
+  <collision>
+    <origin xyz="0.007269 -0.037678 -0.343728" rpy="0 0 0"/>
+    <geometry>
+      <mesh filename="package://dexhand_description/meshes/index-plp_1.stl" scale="0.001 0.001 0.001"/>
+    </geometry>
+  </collision>
+</link>
+<link name="index-mlp_1">
+  <inertial>
+    <origin xyz="-0.0014672452336520862 -0.004861924263139264 0.014904028884496323" rpy="0 0 0"/>
+    <mass value="0.017288956361389173"/>
+    <inertia ixx="1e-06" iyy="1e-06" izz="0.0" ixy="-0.0" iyz="-0.0" ixz="-0.0"/>
+  </inertial>
+  <visual>
+    <origin xyz="0.011959 -0.038935 -0.388702" rpy="0 0 0"/>
+    <geometry>
+      <mesh filename="package://dexhand_description/meshes/index-mlp_1.stl" scale="0.001 0.001 0.001"/>
+    </geometry>
+    <material name="silver"/>
+  </visual>
+  <collision>
+    <origin xyz="0.011959 -0.038935 -0.388702" rpy="0 0 0"/>
+    <geometry>
+      <mesh filename="package://dexhand_description/meshes/index-mlp_1.stl" scale="0.001 0.001 0.001"/>
+    </geometry>
+  </collision>
+</link>
+<link name="index-tip_1">
+  <inertial>
+    <origin xyz="-0.000864193964734649 -0.005385771025884167 0.006769569897979166" rpy="0 0 0"/>
+    <mass value="0.0160783570939756"/>
+    <inertia ixx="1e-06" iyy="1e-06" izz="0.0" ixy="-0.0" iyz="-0.0" ixz="0.0"/>
+  </inertial>
+  <visual>
+    <origin xyz="0.013327 -0.041154 -0.418589" rpy="0 0 0"/>
+    <geometry>
+      <mesh filename="package://dexhand_description/meshes/index-tip_1.stl" scale="0.001 0.001 0.001"/>
+    </geometry>
+    <material name="silver"/>
+  </visual>
+  <collision>
+    <origin xyz="0.013327 -0.041154 -0.418589" rpy="0 0 0"/>
+    <geometry>
+      <mesh filename="package://dexhand_description/meshes/index-tip_1.stl" scale="0.001 0.001 0.001"/>
+    </geometry>
+  </collision>
+</link>
+<link name="pinky-bulk_1">
+  <inertial>
+    <origin xyz="0.0027271468848747375 -0.00919661076399992 0.036410887836454076" rpy="0 0 0"/>
+    <mass value="0.11417768838788588"/>
+    <inertia ixx="0.000111" iyy="0.000112" izz="1e-05" ixy="1e-06" iyz="1.3e-05" ixz="-1e-05"/>
+  </inertial>
+  <visual>
+    <origin xyz="0.01198 0.0217 -0.255266" rpy="0 0 0"/>
+    <geometry>
+      <mesh filename="package://dexhand_description/meshes/pinky-bulk_1.stl" scale="0.001 0.001 0.001"/>
+    </geometry>
+    <material name="silver"/>
+  </visual>
+  <collision>
+    <origin xyz="0.01198 0.0217 -0.255266" rpy="0 0 0"/>
+    <geometry>
+      <mesh filename="package://dexhand_description/meshes/pinky-bulk_1.stl" scale="0.001 0.001 0.001"/>
+    </geometry>
+  </collision>
+</link>
+<link name="middle-plp_1">
+  <inertial>
+    <origin xyz="-0.005943581040544219 -0.008199991640619155 0.023732107441142736" rpy="0 0 0"/>
+    <mass value="0.05600912510930776"/>
+    <inertia ixx="1.3e-05" iyy="1.3e-05" izz="2e-06" ixy="0.0" iyz="0.0" ixz="0.0"/>
+  </inertial>
+  <visual>
+    <origin xyz="0.007096 -0.0143 -0.350266" rpy="0 0 0"/>
+    <geometry>
+      <mesh filename="package://dexhand_description/meshes/middle-plp_1.stl" scale="0.001 0.001 0.001"/>
+    </geometry>
+    <material name="silver"/>
+  </visual>
+  <collision>
+    <origin xyz="0.007096 -0.0143 -0.350266" rpy="0 0 0"/>
+    <geometry>
+      <mesh filename="package://dexhand_description/meshes/middle-plp_1.stl" scale="0.001 0.001 0.001"/>
+    </geometry>
+  </collision>
+</link>
+<link name="middle-mlp_1">
+  <inertial>
+    <origin xyz="-0.0002942937668230297 -0.006300032078833903 0.01528820861860325" rpy="0 0 0"/>
+    <mass value="0.019660714741942815"/>
+    <inertia ixx="1e-06" iyy="1e-06" izz="1e-06" ixy="0.0" iyz="0.0" ixz="-0.0"/>
+  </inertial>
+  <visual>
+    <origin xyz="0.011096 -0.0123 -0.397516" rpy="0 0 0"/>
+    <geometry>
+      <mesh filename="package://dexhand_description/meshes/middle-mlp_1.stl" scale="0.001 0.001 0.001"/>
+    </geometry>
+    <material name="silver"/>
+  </visual>
+  <collision>
+    <origin xyz="0.011096 -0.0123 -0.397516" rpy="0 0 0"/>
+    <geometry>
+      <mesh filename="package://dexhand_description/meshes/middle-mlp_1.stl" scale="0.001 0.001 0.001"/>
+    </geometry>
+  </collision>
+</link>
+<link name="middle-tip_1">
+  <inertial>
+    <origin xyz="-0.0006361624064091121 -0.006200060330852967 0.006854700140433545" rpy="0 0 0"/>
+    <mass value="0.0177222165691614"/>
+    <inertia ixx="1e-06" iyy="1e-06" izz="0.0" ixy="0.0" iyz="0.0" ixz="0.0"/>
+  </inertial>
+  <visual>
+    <origin xyz="0.011096 -0.0123 -0.429016" rpy="0 0 0"/>
+    <geometry>
+      <mesh filename="package://dexhand_description/meshes/middle-tip_1.stl" scale="0.001 0.001 0.001"/>
+    </geometry>
+    <material name="silver"/>
+  </visual>
+  <collision>
+    <origin xyz="0.011096 -0.0123 -0.429016" rpy="0 0 0"/>
+    <geometry>
+      <mesh filename="package://dexhand_description/meshes/middle-tip_1.stl" scale="0.001 0.001 0.001"/>
+    </geometry>
+  </collision>
+</link>
+<link name="ring-plp_1">
+  <inertial>
+    <origin xyz="-0.004988778025381063 -0.011235452676283272 0.021431089299078554" rpy="0 0 0"/>
+    <mass value="0.051607390430851795"/>
+    <inertia ixx="1.1e-05" iyy="1.1e-05" izz="2e-06" ixy="0.0" iyz="1e-06" ixz="-0.0"/>
+  </inertial>
+  <visual>
+    <origin xyz="0.006914 0.010213 -0.347254" rpy="0 0 0"/>
+    <geometry>
+      <mesh filename="package://dexhand_description/meshes/ring-plp_1.stl" scale="0.001 0.001 0.001"/>
+    </geometry>
+    <material name="silver"/>
+  </visual>
+  <collision>
+    <origin xyz="0.006914 0.010213 -0.347254" rpy="0 0 0"/>
+    <geometry>
+      <mesh filename="package://dexhand_description/meshes/ring-plp_1.stl" scale="0.001 0.001 0.001"/>
+    </geometry>
+  </collision>
+</link>
+<link name="ring-mlp_1">
+  <inertial>
+    <origin xyz="0.0003732140836782156 -0.00764471336941365 0.013759338633879348" rpy="0 0 0"/>
+    <mass value="0.017289443732746056"/>
+    <inertia ixx="1e-06" iyy="1e-06" izz="0.0" ixy="0.0" iyz="0.0" ixz="-0.0"/>
+  </inertial>
+  <visual>
+    <origin xyz="0.010293 0.018042 -0.39168" rpy="0 0 0"/>
+    <geometry>
+      <mesh filename="package://dexhand_description/meshes/ring-mlp_1.stl" scale="0.001 0.001 0.001"/>
+    </geometry>
+    <material name="silver"/>
+  </visual>
+  <collision>
+    <origin xyz="0.010293 0.018042 -0.39168" rpy="0 0 0"/>
+    <geometry>
+      <mesh filename="package://dexhand_description/meshes/ring-mlp_1.stl" scale="0.001 0.001 0.001"/>
+    </geometry>
+  </collision>
+</link>
+<link name="ring-tip_1">
+  <inertial>
+    <origin xyz="-2.4752226243757516e-05 -0.006623152446546366 0.00561604826201334" rpy="0 0 0"/>
+    <mass value="0.016038982608931798"/>
+    <inertia ixx="1e-06" iyy="1e-06" izz="0.0" ixy="0.0" iyz="0.0" ixz="0.0"/>
+  </inertial>
+  <visual>
+    <origin xyz="0.010021 0.021513 -0.421477" rpy="0 0 0"/>
+    <geometry>
+      <mesh filename="package://dexhand_description/meshes/ring-tip_1.stl" scale="0.001 0.001 0.001"/>
+    </geometry>
+    <material name="silver"/>
+  </visual>
+  <collision>
+    <origin xyz="0.010021 0.021513 -0.421477" rpy="0 0 0"/>
+    <geometry>
+      <mesh filename="package://dexhand_description/meshes/ring-tip_1.stl" scale="0.001 0.001 0.001"/>
+    </geometry>
+  </collision>
+</link>
+<link name="pinky-plp_1">
+  <inertial>
+    <origin xyz="-0.003810668938620476 -0.012545146418320559 0.01824146705849028" rpy="0 0 0"/>
+    <mass value="0.04272741599660885"/>
+    <inertia ixx="8e-06" iyy="8e-06" izz="1e-06" ixy="0.0" iyz="1e-06" ixz="-0.0"/>
+  </inertial>
+  <visual>
+    <origin xyz="0.007304 0.030405 -0.339487" rpy="0 0 0"/>
+    <geometry>
+      <mesh filename="package://dexhand_description/meshes/pinky-plp_1.stl" scale="0.001 0.001 0.001"/>
+    </geometry>
+    <material name="silver"/>
+  </visual>
+  <collision>
+    <origin xyz="0.007304 0.030405 -0.339487" rpy="0 0 0"/>
+    <geometry>
+      <mesh filename="package://dexhand_description/meshes/pinky-plp_1.stl" scale="0.001 0.001 0.001"/>
+    </geometry>
+  </collision>
+</link>
+<link name="pinky-mlp_1">
+  <inertial>
+    <origin xyz="0.001048124969384794 -0.00753053358362181 0.011942260100064106" rpy="0 0 0"/>
+    <mass value="0.012979924052628225"/>
+    <inertia ixx="1e-06" iyy="1e-06" izz="0.0" ixy="0.0" iyz="0.0" ixz="-0.0"/>
+  </inertial>
+  <visual>
+    <origin xyz="0.009816 0.040989 -0.37881" rpy="0 0 0"/>
+    <geometry>
+      <mesh filename="package://dexhand_description/meshes/pinky-mlp_1.stl" scale="0.001 0.001 0.001"/>
+    </geometry>
+    <material name="silver"/>
+  </visual>
+  <collision>
+    <origin xyz="0.009816 0.040989 -0.37881" rpy="0 0 0"/>
+    <geometry>
+      <mesh filename="package://dexhand_description/meshes/pinky-mlp_1.stl" scale="0.001 0.001 0.001"/>
+    </geometry>
+  </collision>
+</link>
+<link name="pinky-tip_1">
+  <inertial>
+    <origin xyz="0.0005692184398215418 -0.006140261264943145 0.004252021497514635" rpy="0 0 0"/>
+    <mass value="0.012880734939160096"/>
+    <inertia ixx="1e-06" iyy="1e-06" izz="0.0" ixy="0.0" iyz="0.0" ixz="0.0"/>
+  </inertial>
+  <visual>
+    <origin xyz="0.009341 0.045675 -0.405396" rpy="0 0 0"/>
+    <geometry>
+      <mesh filename="package://dexhand_description/meshes/pinky-tip_1.stl" scale="0.001 0.001 0.001"/>
+    </geometry>
+    <material name="silver"/>
+  </visual>
+  <collision>
+    <origin xyz="0.009341 0.045675 -0.405396" rpy="0 0 0"/>
+    <geometry>
+      <mesh filename="package://dexhand_description/meshes/pinky-tip_1.stl" scale="0.001 0.001 0.001"/>
     </geometry>
   </collision>
@@ -273,9 +513,4 @@
   <child link="middle-bulk_1"/>
 </joint>
-<joint name="pinky-bulk" type="fixed">
-  <origin xyz="2e-05 -0.0217 0.255266" rpy="0 0 0"/>
-  <parent link="wrist-upper_1"/>
-  <child link="pinky-bulk_1"/>
-</joint>
 <joint name="ring-bulk" type="fixed">
   <origin xyz="0.0 -0.029 0.0" rpy="0 0 0"/>
@@ -305,5 +540,5 @@
 </joint>
 <joint name="pinky-yaw" type="revolute">
-  <origin xyz="0.010544 -0.017545 -0.153237" rpy="0 0 0"/>
+  <origin xyz="-0.001436 -0.017245 0.078763" rpy="0 0 0"/>
   <parent link="pinky-bulk_1"/>
   <child link="pinky-knuckle_1"/>
@@ -311,3 +546,92 @@
   <limit upper="0.349066" lower="-0.349066" effort="100" velocity="100"/>
 </joint>
+<joint name="index-pitch" type="revolute">
+  <origin xyz="0.008616 0.007539 0.003571" rpy="0 0 0"/>
+  <parent link="index-knuckle_1"/>
+  <child link="index-plp_1"/>
+  <axis xyz="0.087977 0.993678 -0.069746"/>
+  <limit upper="0.785398" lower="0.0" effort="100" velocity="100"/>
+</joint>
+<joint name="index-knuckle" type="revolute">
+  <origin xyz="-0.00469 0.001257 0.044974" rpy="0 0 0"/>
+  <parent link="index-plp_1"/>
+  <child link="index-mlp_1"/>
+  <axis xyz="0.087977 0.993678 -0.069746"/>
+  <limit upper="0.785398" lower="0.0" effort="100" velocity="100"/>
+</joint>
+<joint name="index-tip" type="revolute">
+  <origin xyz="-0.001368 0.002219 0.029887" rpy="0 0 0"/>
+  <parent link="index-mlp_1"/>
+  <child link="index-tip_1"/>
+  <axis xyz="0.087977 0.993678 -0.069746"/>
+  <limit upper="0.785398" lower="0.0" effort="100" velocity="100"/>
+</joint>
+<joint name="pinky-bulk" type="fixed">
+  <origin xyz="0.012 -0.021 0.023266" rpy="0 0 0"/>
+  <parent link="wrist-upper_1"/>
+  <child link="pinky-bulk_1"/>
+</joint>
+<joint name="middle-pitch" type="revolute">
+  <origin xyz="0.00775 0.008 0.004" rpy="0 0 0"/>
+  <parent link="middle-knuckle_1"/>
+  <child link="middle-plp_1"/>
+  <axis xyz="0.0 1.0 0.0"/>
+  <limit upper="0.785398" lower="0.0" effort="100" velocity="100"/>
+</joint>
+<joint name="middle-knuckle" type="revolute">
+  <origin xyz="-0.004 -0.002 0.04725" rpy="0 0 0"/>
+  <parent link="middle-plp_1"/>
+  <child link="middle-mlp_1"/>
+  <axis xyz="-0.0 1.0 0.0"/>
+  <limit upper="0.785398" lower="0.0" effort="100" velocity="100"/>
+</joint>
+<joint name="middle-tip" type="revolute">
+  <origin xyz="0.0 0.0 0.0315" rpy="0 0 0"/>
+  <parent link="middle-mlp_1"/>
+  <child link="middle-tip_1"/>
+  <axis xyz="-0.0 1.0 0.0"/>
+  <limit upper="0.785398" lower="0.0" effort="100" velocity="100"/>
+</joint>
+<joint name="ring-pitch" type="revolute">
+  <origin xyz="0.007067 0.008125 0.004909" rpy="0 0 0"/>
+  <parent link="ring-knuckle_1"/>
+  <child link="ring-plp_1"/>
+  <axis xyz="-0.086225 0.989495 0.116038"/>
+  <limit upper="0.785398" lower="0.0" effort="100" velocity="100"/>
+</joint>
+<joint name="ring-knuckle" type="revolute">
+  <origin xyz="-0.003379 -0.007829 0.044426" rpy="0 0 0"/>
+  <parent link="ring-plp_1"/>
+  <child link="ring-mlp_1"/>
+  <axis xyz="-0.086225 0.989495 0.116038"/>
+  <limit upper="0.785398" lower="0.0" effort="100" velocity="100"/>
+</joint>
+<joint name="ring-tip" type="revolute">
+  <origin xyz="0.000272 -0.003471 0.029797" rpy="0 0 0"/>
+  <parent link="ring-mlp_1"/>
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
Commit message: Added in thumb - all DOF's present

File: urdf/dexhand.xacro (robot description, xacro)
@@ -484,4 +484,104 @@
   </collision>
 </link>
+<link name="thumb-cmc-b_1">
+  <inertial>
+    <origin xyz="0.003351252729851968 0.0058106071637870765 -0.00814154865248179" rpy="0 0 0"/>
+    <mass value="0.008494087027059793"/>
+    <inertia ixx="0.0" iyy="0.0" izz="0.0" ixy="-0.0" iyz="0.0" ixz="0.0"/>
+  </inertial>
+  <visual>
+    <origin xyz="-0.014937 -0.01879 -0.268001" rpy="0 0 0"/>
+    <geometry>
+      <mesh filename="package://dexhand_description/meshes/thumb-cmc-b_1.stl" scale="0.001 0.001 0.001"/>
+    </geometry>
+    <material name="silver"/>
+  </visual>
+  <collision>
+    <origin xyz="-0.014937 -0.01879 -0.268001" rpy="0 0 0"/>
+    <geometry>
+      <mesh filename="package://dexhand_description/meshes/thumb-cmc-b_1.stl" scale="0.001 0.001 0.001"/>
+    </geometry>
+  </collision>
+</link>
+<link name="thumb-cmc-a_1">
+  <inertial>
+    <origin xyz="0.002946681038430113 0.005054293341482705 0.005851296597689182" rpy="0 0 0"/>
+    <mass value="0.015039242610946097"/>
+    <inertia ixx="0.0" iyy="0.0" izz="0.0" ixy="0.0" iyz="-0.0" ixz="-0.0"/>
+  </inertial>
+  <visual>
+    <origin xyz="-0.017759 -0.023693 -0.258808" rpy="0 0 0"/>
+    <geometry>
+      <mesh filename="package://dexhand_description/meshes/thumb-cmc-a_1.stl" scale="0.001 0.001 0.001"/>
+    </geometry>
+    <material name="silver"/>
+  </visual>
+  <collision>
+    <origin xyz="-0.017759 -0.023693 -0.258808" rpy="0 0 0"/>
+    <geometry>
+      <mesh filename="package://dexhand_description/meshes/thumb-cmc-a_1.stl" scale="0.001 0.001 0.001"/>
+    </geometry>
+  </collision>
+</link>
+<link name="thumb-plp_1">
+  <inertial>
+    <origin xyz="0.005433746290735175 0.025637034957291676 0.016614706566931703" rpy="0 0 0"/>
+    <mass value="0.06710748615776632"/>
+    <inertia ixx="2e-05" iyy="1.5e-05" izz="1.3e-05" ixy="-5e-06" iyz="-9e-06" ixz="-5e-06"/>
+  </inertial>
+  <visual>
+    <origin xyz="-0.028683 -0.026348 -0.26657" rpy="0 0 0"/>
+    <geometry>
+      <mesh filename="package://dexhand_description/meshes/thumb-plp_1.stl" scale="0.001 0.001 0.001"/>
+    </geometry>
+    <material name="silver"/>
+  </visual>
+  <collision>
+    <origin xyz="-0.028683 -0.026348 -0.26657" rpy="0 0 0"/>
+    <geometry>
+      <mesh filename="package://dexhand_description/meshes/thumb-plp_1.stl" scale="0.001 0.001 0.001"/>
+    </geometry>
+  </collision>
+</link>
+<link name="thumb-mlp_1">
+  <inertial>
+    <origin xyz="0.002151568364903572 0.015611380274394515 0.012743956202626694" rpy="0 0 0"/>
+    <mass value="0.025187203449803457"/>
+    <inertia ixx="2e-06" iyy="2e-06" izz="2e-06" ixy="-0.0" iyz="-1e-06" ixz="-0.0"/>
+  </inertial>
+  <visual>
+    <origin xyz="-0.049475 -0.066604 -0.306172" rpy="0 0 0"/>
+    <geometry>
+      <mesh filename="package://dexhand_description/meshes/thumb-mlp_1.stl" scale="0.001 0.001 0.001"/>
+    </geometry>
+    <material name="silver"/>
+  </visual>
+  <collision>
+    <origin xyz="-0.049475 -0.066604 -0.306172" rpy="0 0 0"/>
+    <geometry>
+      <mesh filename="package://dexhand_description/meshes/thumb-mlp_1.stl" scale="0.001 0.001 0.001"/>
+    </geometry>
+  </collision>
+</link>
+<link name="thumb-tip_1">
+  <inertial>
+    <origin xyz="-0.0009246362325292662 0.010131321702323684 0.007474037055237581" rpy="0 0 0"/>
+    <mass value="0.02316990761545859"/>
+    <inertia ixx="2e-06" iyy="2e-06" izz="2e-06" ixy="-0.0" iyz="-1e-06" ixz="-0.0"/>
+  </inertial>
+  <visual>
+    <origin xyz="-0.064312 -0.092065 -0.333221" rpy="0 0 0"/>
+    <geometry>
+      <mesh filename="package://dexhand_description/meshes/thumb-tip_1.stl" scale="0.001 0.001 0.001"/>
+    </geometry>
+    <material name="silver"/>
+  </visual>
+  <collision>
+    <origin xyz="-0.064312 -0.092065 -0.333221" rpy="0 0 0"/>
+    <geometry>
+      <mesh filename="package://dexhand_description/meshes/thumb-tip_1.stl" scale="0.001 0.001 0.001"/>
+    </geometry>
+  </collision>
+</link>
 <joint name="flange" type="fixed">
   <origin xyz="0.0 0.0 0.0" rpy="0 0 0"/>
@@ -635,3 +735,38 @@
   <limit upper="0.785398" lower="0.0" effort="100" velocity="100"/>
 </joint>
+<joint name="thumb-yaw" type="revolute">
+  <origin xyz="0.026917 -0.00751 0.012735" rpy="0 0 0"/>
+  <parent link="middle-bulk_1"/>
+  <child link="thumb-cmc-b_1"/>
+  <axis xyz="0.353553 0.612372 -0.707107"/>
+  <limit upper="0.872665" lower="0.0" effort="100" velocity="100"/>
+</joint>
+<joint name="thumb-roll" type="revolute">
+  <origin xyz="0.002822 0.004903 -0.009193" rpy="0 0 0"/>
+  <parent link="thumb-cmc-b_1"/>
+  <child link="thumb-cmc-a_1"/>
+  <axis xyz="-0.35613 -0.610881 -0.707104"/>
+  <limit upper="0.349066" lower="0.0" effort="100" velocity="100"/>
+</joint>
+<joint name="thumb-pitch" type="revolute">
+  <origin xyz="0.010924 0.002655 0.007762" rpy="0 0 0"/>
+  <parent link="thumb-cmc-a_1"/>
+  <child link="thumb-plp_1"/>
+  <axis xyz="0.864969 -0.501821 -0.002105"/>
+  <limit upper="1.047198" lower="0.0" effort="100" velocity="100"/>
+</joint>
+<joint name="thumb-knuckle" type="revolute">
+  <origin xyz="0.020792 0.040256 0.039602" rpy="0 0 0"/>
+  <parent link="thumb-plp_1"/>
+  <child link="thumb-mlp_1"/>
+  <axis xyz="0.864969 -0.501821 -0.002105"/>
+  <limit upper="0.785398" lower="0.0" effort="100" velocity="100"/>
+</joint>
+<joint name="thumb-tip" type="revolute">
+  <origin xyz="0.014837 0.025461 0.027049" rpy="0 0 0"/>
+  <parent link="thumb-mlp_1"/>
+  <child link="thumb-tip_1"/>
+  <axis xyz="0.864969 -0.501821 -0.002105"/>
+  <limit upper="0.785398" lower="0.0" effort="100" velocity="100"/>
+</joint>
 </robot>
