Commit message: Unified naming convention around underscores

File: urdf/dexhand.xacro (robot description, xacro)
@@ -44,5 +44,5 @@
   </collision>
 </link>
-<link name="wrist-lower_1">
+<link name="wrist_lower_1">
   <inertial>
     <origin xyz="-3.0683763790256835e-05 0.02099365535807374 0.021635071099651598" rpy="0 0 0"/>
@@ -53,5 +53,5 @@
     <origin xyz="0.012 0.0217 -0.203" rpy="0 0 0"/>
     <geometry>
-      <mesh filename="package://dexhand_description/meshes/wrist-lower_1.stl" scale="0.001 0.001 0.001"/>
+      <mesh filename="package://dexhand_description/meshes/wrist_lower_1.stl" scale="0.001 0.001 0.001"/>
     </geometry>
     <material name="silver"/>
@@ -60,9 +60,9 @@
     <origin xyz="0.012 0.0217 -0.203" rpy="0 0 0"/>
     <geometry>
-      <mesh filename="package://dexhand_description/meshes/wrist-lower_1.stl" scale="0.001 0.001 0.001"/>
-    </geometry>
-  </collision>
-</link>
-<link name="wrist-upper_1">
+      <mesh filename="package://dexhand_description/meshes/wrist_lower_1.stl" scale="0.001 0.001 0.001"/>
+    </geometry>
+  </collision>
+</link>
+<link name="wrist_upper_1">
   <inertial>
     <origin xyz="0.011943478530919125 1.976395235870395e-08 0.007146961841600852" rpy="0 0 0"/>
@@ -73,5 +73,5 @@
     <origin xyz="0.02398 0.0007 -0.232" rpy="0 0 0"/>
     <geometry>
-      <mesh filename="package://dexhand_description/meshes/wrist-upper_1.stl" scale="0.001 0.001 0.001"/>
+      <mesh filename="package://dexhand_description/meshes/wrist_upper_1.stl" scale="0.001 0.001 0.001"/>
     </geometry>
     <material name="silver"/>
@@ -80,9 +80,9 @@
     <origin xyz="0.02398 0.0007 -0.232" rpy="0 0 0"/>
     <geometry>
-      <mesh filename="package://dexhand_description/meshes/wrist-upper_1.stl" scale="0.001 0.001 0.001"/>
-    </geometry>
-  </collision>
-</link>
-<link name="index-bulk_1">
+      <mesh filename="package://dexhand_description/meshes/wrist_upper_1.stl" scale="0.001 0.001 0.001"/>
+    </geometry>
+  </collision>
+</link>
+<link name="index_bulk_1">
   <inertial>
     <origin xyz="0.001953836875769263 0.005732502869548333 0.04310739786858114" rpy="0 0 0"/>
@@ -93,5 +93,5 @@
     <origin xyz="0.01198 -0.0203 -0.255266" rpy="0 0 0"/>
     <geometry>
-      <mesh filename="package://dexhand_description/meshes/index-bulk_1.stl" scale="0.001 0.001 0.001"/>
+      <mesh filename="package://dexhand_description/meshes/index_bulk_1.stl" scale="0.001 0.001 0.001"/>
     </geometry>
     <material name="silver"/>
@@ -100,9 +100,9 @@
     <origin xyz="0.01198 -0.0203 -0.255266" rpy="0 0 0"/>
     <geometry>
-      <mesh filename="package://dexhand_description/meshes/index-bulk_1.stl" scale="0.001 0.001 0.001"/>
-    </geometry>
-  </collision>
-</link>
-<link name="middle-bulk_1">
+      <mesh filename="package://dexhand_description/meshes/index_bulk_1.stl" scale="0.001 0.001 0.001"/>
+    </geometry>
+  </collision>
+</link>
+<link name="middle_bulk_1">
   <inertial>
     <origin xyz="0.01064695002640492 -0.0158135798135519 0.030689623412746947" rpy="0 0 0"/>
@@ -113,5 +113,5 @@
     <origin xyz="0.01198 -0.0263 -0.255266" rpy="0 0 0"/>
     <geometry>
-      <mesh filename="package://dexhand_description/meshes/middle-bulk_1.stl" scale="0.001 0.001 0.001"/>
+      <mesh filename="package://dexhand_description/meshes/middle_bulk_1.stl" scale="0.001 0.001 0.001"/>
     </geometry>
     <material name="silver"/>
@@ -120,9 +120,9 @@
     <origin xyz="0.01198 -0.0263 -0.255266" rpy="0 0 0"/>
     <geometry>
-      <mesh filename="package://dexhand_description/meshes/middle-bulk_1.stl" scale="0.001 0.001 0.001"/>
-    </geometry>
-  </collision>
-</link>
-<link name="ring-bulk_1">
+      <mesh filename="package://dexhand_description/meshes/middle_bulk_1.stl" scale="0.001 0.001 0.001"/>
+    </geometry>
+  </collision>
+</link>
+<link name="ring_bulk_1">
   <inertial>
     <origin xyz="0.003391811603104285 -0.01025124324374128 0.05277806405684754" rpy="0 0 0"/>
@@ -133,5 +133,5 @@
     <origin xyz="0.01198 0.0027 -0.255266" rpy="0 0 0"/>
     <geometry>
-      <mesh filename="package://dexhand_description/meshes/ring-bulk_1.stl" scale="0.001 0.001 0.001"/>
+      <mesh filename="package://dexhand_description/meshes/ring_bulk_1.stl" scale="0.001 0.001 0.001"/>
     </geometry>
     <material name="silver"/>
@@ -140,9 +140,9 @@
     <origin xyz="0.01198 0.0027 -0.255266" rpy="0 0 0"/>
     <geometry>
-      <mesh filename="package://dexhand_description/meshes/ring-bulk_1.stl" scale="0.001 0.001 0.001"/>
-    </geometry>
-  </collision>
-</link>
-<link name="index-knuckle_1">
+      <mesh filename="package://dexhand_description/meshes/ring_bulk_1.stl" scale="0.001 0.001 0.001"/>
+    </geometry>
+  </collision>
+</link>
+<link name="index_knuckle_1">
   <inertial>
     <origin xyz="0.007134673083101478 -0.0005540875413111747 0.0011013348331220807" rpy="0 0 0"/>
@@ -153,5 +153,5 @@
     <origin xyz="0.015885 -0.030139 -0.340157" rpy="0 0 0"/>
     <geometry>
-      <mesh filename="package://dexhand_description/meshes/index-knuckle_1.stl" scale="0.001 0.001 0.001"/>
+      <mesh filename="package://dexhand_description/meshes/index_knuckle_1.stl" scale="0.001 0.001 0.001"/>
     </geometry>
     <material name="silver"/>
@@ -160,9 +160,9 @@
     <origin xyz="0.015885 -0.030139 -0.340157" rpy="0 0 0"/>
     <geometry>
-      <mesh filename="package://dexhand_description/meshes/index-knuckle_1.stl" scale="0.001 0.001 0.001"/>
-    </geometry>
-  </collision>
-</link>
-<link name="middle-knuckle_1">
+      <mesh filename="package://dexhand_description/meshes/index_knuckle_1.stl" scale="0.001 0.001 0.001"/>
+    </geometry>
+  </collision>
+</link>
+<link name="middle_knuckle_1">
   <inertial>
     <origin xyz="0.006935399474227782 3.095281810635425e-08 0.0009794888636300847" rpy="0 0 0"/>
@@ -173,5 +173,5 @@
     <origin xyz="0.014846 -0.0063 -0.346266" rpy="0 0 0"/>
     <geometry>
-      <mesh filename="package://dexhand_description/meshes/middle-knuckle_1.stl" scale="0.001 0.001 0.001"/>
+      <mesh filename="package://dexhand_description/meshes/middle_knuckle_1.stl" scale="0.001 0.001 0.001"/>
     </geometry>
     <material name="silver"/>
@@ -180,9 +180,9 @@
     <origin xyz="0.014846 -0.0063 -0.346266" rpy="0 0 0"/>
     <geometry>
-      <mesh filename="package://dexhand_description/meshes/middle-knuckle_1.stl" scale="0.001 0.001 0.001"/>
-    </geometry>
-  </collision>
-</link>
-<link name="ring-knuckle_1">
+      <mesh filename="package://dexhand_description/meshes/middle_knuckle_1.stl" scale="0.001 0.001 0.001"/>
+    </geometry>
+  </collision>
+</link>
+<link name="ring_knuckle_1">
   <inertial>
     <origin xyz="0.006918049206992894 0.0004875294278836907 0.0009797412002323647" rpy="0 0 0"/>
@@ -193,5 +193,5 @@
     <origin xyz="0.013981 0.018338 -0.342345" rpy="0 0 0"/>
     <geometry>
-      <mesh filename="package://dexhand_description/meshes/ring-knuckle_1.stl" scale="0.001 0.001 0.001"/>
+      <mesh filename="package://dexhand_description/meshes/ring_knuckle_1.stl" scale="0.001 0.001 0.001"/>
     </geometry>
     <material name="silver"/>
@@ -200,9 +200,9 @@
     <origin xyz="0.013981 0.018338 -0.342345" rpy="0 0 0"/>
     <geometry>
-      <mesh filename="package://dexhand_description/meshes/ring-knuckle_1.stl" scale="0.001 0.001 0.001"/>
-    </geometry>
-  </collision>
-</link>
-<link name="pinky-knuckle_1">
+      <mesh filename="package://dexhand_description/meshes/ring_knuckle_1.stl" scale="0.001 0.001 0.001"/>
+    </geometry>
+  </collision>
+</link>
+<link name="pinky_knuckle_1">
   <inertial>
     <origin xyz="0.006818820473942549 0.0011824337110899266 0.0010801856787569508" rpy="0 0 0"/>
@@ -213,5 +213,5 @@
     <origin xyz="0.013416 0.038945 -0.334029" rpy="0 0 0"/>
     <geometry>
-      <mesh filename="package://dexhand_description/meshes/pinky-knuckle_1.stl" scale="0.001 0.001 0.001"/>
+      <mesh filename="package://dexhand_description/meshes/pinky_knuckle_1.stl" scale="0.001 0.001 0.001"/>
     </geometry>
     <material name="silver"/>
@@ -220,9 +220,9 @@
     <origin xyz="0.013416 0.038945 -0.334029" rpy="0 0 0"/>
     <geometry>
-      <mesh filename="package://dexhand_description/meshes/pinky-knuckle_1.stl" scale="0.001 0.001 0.001"/>
-    </geometry>
-  </collision>
-</link>
-<link name="index-plp_1">
+      <mesh filename="package://dexhand_description/meshes/pinky_knuckle_1.stl" scale="0.001 0.001 0.001"/>
+    </geometry>
+  </collision>
+</link>
+<link name="index_plp_1">
   <inertial>
     <origin xyz="-0.006869198158126709 -0.006033909809302199 0.022940465298997237" rpy="0 0 0"/>
@@ -233,5 +233,5 @@
     <origin xyz="0.007269 -0.037678 -0.343728" rpy="0 0 0"/>
     <geometry>
-      <mesh filename="package://dexhand_description/meshes/index-plp_1.stl" scale="0.001 0.001 0.001"/>
+      <mesh filename="package://dexhand_description/meshes/index_plp_1.stl" scale="0.001 0.001 0.001"/>
     </geometry>
     <material name="silver"/>
@@ -240,9 +240,9 @@
     <origin xyz="0.007269 -0.037678 -0.343728" rpy="0 0 0"/>
     <geometry>
-      <mesh filename="package://dexhand_description/meshes/index-plp_1.stl" scale="0.001 0.001 0.001"/>
-    </geometry>
-  </collision>
-</link>
-<link name="index-mlp_1">
+      <mesh filename="package://dexhand_description/meshes/index_plp_1.stl" scale="0.001 0.001 0.001"/>
+    </geometry>
+  </collision>
+</link>
+<link name="index_mlp_1">
   <inertial>
     <origin xyz="-0.0014672452336520862 -0.004861924263139264 0.014904028884496323" rpy="0 0 0"/>
@@ -253,5 +253,5 @@
     <origin xyz="0.011959 -0.038935 -0.388702" rpy="0 0 0"/>
     <geometry>
-      <mesh filename="package://dexhand_description/meshes/index-mlp_1.stl" scale="0.001 0.001 0.001"/>
+      <mesh filename="package://dexhand_description/meshes/index_mlp_1.stl" scale="0.001 0.001 0.001"/>
     </geometry>
     <material name="silver"/>
@@ -260,9 +260,9 @@
     <origin xyz="0.011959 -0.038935 -0.388702" rpy="0 0 0"/>
     <geometry>
-      <mesh filename="package://dexhand_description/meshes/index-mlp_1.stl" scale="0.001 0.001 0.001"/>
-    </geometry>
-  </collision>
-</link>
-<link name="index-tip_1">
+      <mesh filename="package://dexhand_description/meshes/index_mlp_1.stl" scale="0.001 0.001 0.001"/>
+    </geometry>
+  </collision>
+</link>
+<link name="index_tip_1">
   <inertial>
     <origin xyz="-0.000864193964734649 -0.005385771025884167 0.006769569897979166" rpy="0 0 0"/>
@@ -273,5 +273,5 @@
     <origin xyz="0.013327 -0.041154 -0.418589" rpy="0 0 0"/>
     <geometry>
-      <mesh filename="package://dexhand_description/meshes/index-tip_1.stl" scale="0.001 0.001 0.001"/>
+      <mesh filename="package://dexhand_description/meshes/index_tip_1.stl" scale="0.001 0.001 0.001"/>
     </geometry>
     <material name="silver"/>
@@ -280,9 +280,9 @@
     <origin xyz="0.013327 -0.041154 -0.418589" rpy="0 0 0"/>
     <geometry>
-      <mesh filename="package://dexhand_description/meshes/index-tip_1.stl" scale="0.001 0.001 0.001"/>
-    </geometry>
-  </collision>
-</link>
-<link name="pinky-bulk_1">
+      <mesh filename="package://dexhand_description/meshes/index_tip_1.stl" scale="0.001 0.001 0.001"/>
+    </geometry>
+  </collision>
+</link>
+<link name="pinky_bulk_1">
   <inertial>
     <origin xyz="0.0027271468848747375 -0.00919661076399992 0.036410887836454076" rpy="0 0 0"/>
@@ -293,5 +293,5 @@
     <origin xyz="0.01198 0.0217 -0.255266" rpy="0 0 0"/>
     <geometry>
-      <mesh filename="package://dexhand_description/meshes/pinky-bulk_1.stl" scale="0.001 0.001 0.001"/>
+      <mesh filename="package://dexhand_description/meshes/pinky_bulk_1.stl" scale="0.001 0.001 0.001"/>
     </geometry>
     <material name="silver"/>
@@ -300,9 +300,9 @@
     <origin xyz="0.01198 0.0217 -0.255266" rpy="0 0 0"/>
     <geometry>
-      <mesh filename="package://dexhand_description/meshes/pinky-bulk_1.stl" scale="0.001 0.001 0.001"/>
-    </geometry>
-  </collision>
-</link>
-<link name="middle-plp_1">
+      <mesh filename="package://dexhand_description/meshes/pinky_bulk_1.stl" scale="0.001 0.001 0.001"/>
+    </geometry>
+  </collision>
+</link>
+<link name="middle_plp_1">
   <inertial>
     <origin xyz="-0.005943581040544219 -0.008199991640619155 0.023732107441142736" rpy="0 0 0"/>
@@ -313,5 +313,5 @@
     <origin xyz="0.007096 -0.0143 -0.350266" rpy="0 0 0"/>
     <geometry>
-      <mesh filename="package://dexhand_description/meshes/middle-plp_1.stl" scale="0.001 0.001 0.001"/>
+      <mesh filename="package://dexhand_description/meshes/middle_plp_1.stl" scale="0.001 0.001 0.001"/>
     </geometry>
     <material name="silver"/>
@@ -320,9 +320,9 @@
     <origin xyz="0.007096 -0.0143 -0.350266" rpy="0 0 0"/>
     <geometry>
-      <mesh filename="package://dexhand_description/meshes/middle-plp_1.stl" scale="0.001 0.001 0.001"/>
-    </geometry>
-  </collision>
-</link>
-<link name="middle-mlp_1">
+      <mesh filename="package://dexhand_description/meshes/middle_plp_1.stl" scale="0.001 0.001 0.001"/>
+    </geometry>
+  </collision>
+</link>
+<link name="middle_mlp_1">
   <inertial>
     <origin xyz="-0.0002942937668230297 -0.006300032078833903 0.01528820861860325" rpy="0 0 0"/>
@@ -333,5 +333,5 @@
     <origin xyz="0.011096 -0.0123 -0.397516" rpy="0 0 0"/>
     <geometry>
-      <mesh filename="package://dexhand_description/meshes/middle-mlp_1.stl" scale="0.001 0.001 0.001"/>
+      <mesh filename="package://dexhand_description/meshes/middle_mlp_1.stl" scale="0.001 0.001 0.001"/>
     </geometry>
     <material name="silver"/>
@@ -340,9 +340,9 @@
     <origin xyz="0.011096 -0.0123 -0.397516" rpy="0 0 0"/>
     <geometry>
-      <mesh filename="package://dexhand_description/meshes/middle-mlp_1.stl" scale="0.001 0.001 0.001"/>
-    </geometry>
-  </collision>
-</link>
-<link name="middle-tip_1">
+      <mesh filename="package://dexhand_description/meshes/middle_mlp_1.stl" scale="0.001 0.001 0.001"/>
+    </geometry>
+  </collision>
+</link>
+<link name="middle_tip_1">
   <inertial>
     <origin xyz="-0.0006361624064091121 -0.006200060330852967 0.006854700140433545" rpy="0 0 0"/>
@@ -353,5 +353,5 @@
     <origin xyz="0.011096 -0.0123 -0.429016" rpy="0 0 0"/>
     <geometry>
-      <mesh filename="package://dexhand_description/meshes/middle-tip_1.stl" scale="0.001 0.001 0.001"/>
+      <mesh filename="package://dexhand_description/meshes/middle_tip_1.stl" scale="0.001 0.001 0.001"/>
     </geometry>
     <material name="silver"/>
@@ -360,9 +360,9 @@
     <origin xyz="0.011096 -0.0123 -0.429016" rpy="0 0 0"/>
     <geometry>
-      <mesh filename="package://dexhand_description/meshes/middle-tip_1.stl" scale="0.001 0.001 0.001"/>
-    </geometry>
-  </collision>
-</link>
-<link name="ring-plp_1">
+      <mesh filename="package://dexhand_description/meshes/middle_tip_1.stl" scale="0.001 0.001 0.001"/>
+    </geometry>
+  </collision>
+</link>
+<link name="ring_plp_1">
   <inertial>
     <origin xyz="-0.004988778025381063 -0.011235452676283272 0.021431089299078554" rpy="0 0 0"/>
@@ -373,5 +373,5 @@
     <origin xyz="0.006914 0.010213 -0.347254" rpy="0 0 0"/>
     <geometry>
-      <mesh filename="package://dexhand_description/meshes/ring-plp_1.stl" scale="0.001 0.001 0.001"/>
+      <mesh filename="package://dexhand_description/meshes/ring_plp_1.stl" scale="0.001 0.001 0.001"/>
     </geometry>
     <material name="silver"/>
@@ -380,9 +380,9 @@
     <origin xyz="0.006914 0.010213 -0.347254" rpy="0 0 0"/>
     <geometry>
-      <mesh filename="package://dexhand_description/meshes/ring-plp_1.stl" scale="0.001 0.001 0.001"/>
-    </geometry>
-  </collision>
-</link>
-<link name="ring-mlp_1">
+      <mesh filename="package://dexhand_description/meshes/ring_plp_1.stl" scale="0.001 0.001 0.001"/>
+    </geometry>
+  </collision>
+</link>
+<link name="ring_mlp_1">
   <inertial>
     <origin xyz="0.0003732140836782156 -0.00764471336941365 0.013759338633879348" rpy="0 0 0"/>
@@ -393,5 +393,5 @@
     <origin xyz="0.010293 0.018042 -0.39168" rpy="0 0 0"/>
     <geometry>
-      <mesh filename="package://dexhand_description/meshes/ring-mlp_1.stl" scale="0.001 0.001 0.001"/>
+      <mesh filename="package://dexhand_description/meshes/ring_mlp_1.stl" scale="0.001 0.001 0.001"/>
     </geometry>
     <material name="silver"/>
@@ -400,9 +400,9 @@
     <origin xyz="0.010293 0.018042 -0.39168" rpy="0 0 0"/>
     <geometry>
-      <mesh filename="package://dexhand_description/meshes/ring-mlp_1.stl" scale="0.001 0.001 0.001"/>
-    </geometry>
-  </collision>
-</link>
-<link name="ring-tip_1">
+      <mesh filename="package://dexhand_description/meshes/ring_mlp_1.stl" scale="0.001 0.001 0.001"/>
+    </geometry>
+  </collision>
+</link>
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