Commit message: Added additional upper wrist joint

File: urdf/dexhand.urdf (robot description, URDF)
Before this commit: robot dexhand, 29 links, 28 joints
Links:
- removed link index-bulk_1
- removed link index-knuckle_1
- removed link index-mlp_1
- removed link index-plp_1
- removed link index-tip_1
- removed link middle-bulk_1
- removed link middle-knuckle_1
- removed link middle-mlp_1
- removed link middle-plp_1
- removed link middle-tip_1
- removed link pinky-bulk_1
- removed link pinky-knuckle_1
- removed link pinky-mlp_1
- removed link pinky-plp_1
- removed link pinky-tip_1
- removed link ring-bulk_1
- removed link ring-knuckle_1
- removed link ring-mlp_1
- removed link ring-plp_1
- removed link ring-tip_1
- removed link thumb-cmc-a_1
- removed link thumb-cmc-b_1
- removed link thumb-mlp_1
- removed link thumb-plp_1
- removed link thumb-tip_1
- removed link wrist-lower_1
- removed link wrist-upper_1
- added link index_bulk_1, mass 0.10571474174321724; collision mesh filename=package://dexhand_description/meshes/index_bulk_1.stl scale=0.001 0.001 0.001; visual mesh filename=package://dexhand_description/meshes/index_bulk_1.stl scale=0.001 0.001 0.001
- added link index_knuckle_1, mass 0.016772407452453803; collision mesh filename=package://dexhand_description/meshes/index_knuckle_1.stl scale=0.001 0.001 0.001; visual mesh filename=package://dexhand_description/meshes/index_knuckle_1.stl scale=0.001 0.001 0.001
- added link index_mlp_1, mass 0.017288956361389173; collision mesh filename=package://dexhand_description/meshes/index_mlp_1.stl scale=0.001 0.001 0.001; visual mesh filename=package://dexhand_description/meshes/index_mlp_1.stl scale=0.001 0.001 0.001
- added link index_plp_1, mass 0.051567105457974535; collision mesh filename=package://dexhand_description/meshes/index_plp_1.stl scale=0.001 0.001 0.001; visual mesh filename=package://dexhand_description/meshes/index_plp_1.stl scale=0.001 0.001 0.001
- added link index_tip_1, mass 0.0160783570939756; collision mesh filename=package://dexhand_description/meshes/index_tip_1.stl scale=0.001 0.001 0.001; visual mesh filename=package://dexhand_description/meshes/index_tip_1.stl scale=0.001 0.001 0.001
- added link middle_bulk_1, mass 0.2319963124821001; collision mesh filename=package://dexhand_description/meshes/middle_bulk_1.stl scale=0.001 0.001 0.001; visual mesh filename=package://dexhand_description/meshes/middle_bulk_1.stl scale=0.001 0.001 0.001
- added link middle_knuckle_1, mass 0.016772407452453803; collision mesh filename=package://dexhand_description/meshes/middle_knuckle_1.stl scale=0.001 0.001 0.001; visual mesh filename=package://dexhand_description/meshes/middle_knuckle_1.stl scale=0.001 0.001 0.001
- added link middle_mlp_1, mass 0.019660714741942815; collision mesh filename=package://dexhand_description/meshes/middle_mlp_1.stl scale=0.001 0.001 0.001; visual mesh filename=package://dexhand_description/meshes/middle_mlp_1.stl scale=0.001 0.001 0.001
- added link middle_plp_1, mass 0.05600912510930776; collision mesh filename=package://dexhand_description/meshes/middle_plp_1.stl scale=0.001 0.001 0.001; visual mesh filename=package://dexhand_description/meshes/middle_plp_1.stl scale=0.001 0.001 0.001
- added link middle_tip_1, mass 0.0177222165691614; collision mesh filename=package://dexhand_description/meshes/middle_tip_1.stl scale=0.001 0.001 0.001; visual mesh filename=package://dexhand_description/meshes/middle_tip_1.stl scale=0.001 0.001 0.001
- added link pinky_bulk_1, mass 0.11417768838788588; collision mesh filename=package://dexhand_description/meshes/pinky_bulk_1.stl scale=0.001 0.001 0.001; visual mesh filename=package://dexhand_description/meshes/pinky_bulk_1.stl scale=0.001 0.001 0.001
- added link pinky_knuckle_1, mass 0.016772407452453803; collision mesh filename=package://dexhand_description/meshes/pinky_knuckle_1.stl scale=0.001 0.001 0.001; visual mesh filename=package://dexhand_description/meshes/pinky_knuckle_1.stl scale=0.001 0.001 0.001
- added link pinky_mlp_1, mass 0.012979924052628225; collision mesh filename=package://dexhand_description/meshes/pinky_mlp_1.stl scale=0.001 0.001 0.001; visual mesh filename=package://dexhand_description/meshes/pinky_mlp_1.stl scale=0.001 0.001 0.001
- added link pinky_plp_1, mass 0.04272741599660885; collision mesh filename=package://dexhand_description/meshes/pinky_plp_1.stl scale=0.001 0.001 0.001; visual mesh filename=package://dexhand_description/meshes/pinky_plp_1.stl scale=0.001 0.001 0.001
- added link pinky_tip_1, mass 0.012880734939160096; collision mesh filename=package://dexhand_description/meshes/pinky_tip_1.stl scale=0.001 0.001 0.001; visual mesh filename=package://dexhand_description/meshes/pinky_tip_1.stl scale=0.001 0.001 0.001
- added link ring_bulk_1, mass 0.09588694429304498; collision mesh filename=package://dexhand_description/meshes/ring_bulk_1.stl scale=0.001 0.001 0.001; visual mesh filename=package://dexhand_description/meshes/ring_bulk_1.stl scale=0.001 0.001 0.001
- added link ring_knuckle_1, mass 0.016772407452453803; collision mesh filename=package://dexhand_description/meshes/ring_knuckle_1.stl scale=0.001 0.001 0.001; visual mesh filename=package://dexhand_description/meshes/ring_knuckle_1.stl scale=0.001 0.001 0.001
- added link ring_mlp_1, mass 0.017289443732746056; collision mesh filename=package://dexhand_description/meshes/ring_mlp_1.stl scale=0.001 0.001 0.001; visual mesh filename=package://dexhand_description/meshes/ring_mlp_1.stl scale=0.001 0.001 0.001
- added link ring_plp_1, mass 0.051607390430851795; collision mesh filename=package://dexhand_description/meshes/ring_plp_1.stl scale=0.001 0.001 0.001; visual mesh filename=package://dexhand_description/meshes/ring_plp_1.stl scale=0.001 0.001 0.001
- added link ring_tip_1, mass 0.016038982608931798; collision mesh filename=package://dexhand_description/meshes/ring_tip_1.stl scale=0.001 0.001 0.001; visual mesh filename=package://dexhand_description/meshes/ring_tip_1.stl scale=0.001 0.001 0.001
- added link thumb_cmc_a_1, mass 0.015039242610946097; collision mesh filename=package://dexhand_description/meshes/thumb_cmc_a_1.stl scale=0.001 0.001 0.001; visual mesh filename=package://dexhand_description/meshes/thumb_cmc_a_1.stl scale=0.001 0.001 0.001
- added link thumb_cmc_b_1, mass 0.008494087027059793; collision mesh filename=package://dexhand_description/meshes/thumb_cmc_b_1.stl scale=0.001 0.001 0.001; visual mesh filename=package://dexhand_description/meshes/thumb_cmc_b_1.stl scale=0.001 0.001 0.001
- added link thumb_mlp_1, mass 0.025187203449803457; collision mesh filename=package://dexhand_description/meshes/thumb_mlp_1.stl scale=0.001 0.001 0.001; visual mesh filename=package://dexhand_description/meshes/thumb_mlp_1.stl scale=0.001 0.001 0.001
- added link thumb_plp_1, mass 0.06710748615776632; collision mesh filename=package://dexhand_description/meshes/thumb_plp_1.stl scale=0.001 0.001 0.001; visual mesh filename=package://dexhand_description/meshes/thumb_plp_1.stl scale=0.001 0.001 0.001
- added link thumb_tip_1, mass 0.02316990761545859; collision mesh filename=package://dexhand_description/meshes/thumb_tip_1.stl scale=0.001 0.001 0.001; visual mesh filename=package://dexhand_description/meshes/thumb_tip_1.stl scale=0.001 0.001 0.001
- added link wrist_lower_1, mass 0.3236409508310491; collision mesh filename=package://dexhand_description/meshes/wrist_lower_1.stl scale=0.001 0.001 0.001; visual mesh filename=package://dexhand_description/meshes/wrist_lower_1.stl scale=0.001 0.001 0.001
- added link wrist_upper_1, mass 0.12131953205677495; collision mesh filename=package://dexhand_description/meshes/wrist_upper_1.stl scale=0.001 0.001 0.001; visual mesh filename=package://dexhand_description/meshes/wrist_upper_1.stl scale=0.001 0.001 0.001
Joints:
- removed joint index-bulk
- removed joint index-knuckle
- removed joint index-pitch
- removed joint index-tip
- removed joint index-yaw
- removed joint middle-bulk
- removed joint middle-knuckle
- removed joint middle-pitch
- removed joint middle-tip
- removed joint middle-yaw
- removed joint pinky-bulk
- removed joint pinky-knuckle
- removed joint pinky-pitch
- removed joint pinky-tip
- removed joint pinky-yaw
- removed joint ring-bulk
- removed joint ring-knuckle
- removed joint ring-pitch
- removed joint ring-tip
- removed joint ring-yaw
- removed joint thumb-knuckle
- removed joint thumb-pitch
- removed joint thumb-roll
- removed joint thumb-tip
- removed joint thumb-yaw
- removed joint wrist_pitch
- added joint Rigid 43: type fixed, parent ring_bulk_1, child pinky_bulk_1, origin xyz=0.0 -0.006043 0.0 rpy=0 0 0
- added joint index_knuckle: type revolute, parent index_plp_1, child index_mlp_1, origin xyz=-0.00469 0.001257 0.044974 rpy=0 0 0, axis 0.087977 0.993678 -0.069746, limit lower=0.0 upper=0.785398 effort=100 velocity=100
- added joint index_pitch: type revolute, parent index_knuckle_1, child index_plp_1, origin xyz=0.008616 0.007539 0.003571 rpy=0 0 0, axis 0.087977 0.993678 -0.069746, limit lower=0.0 upper=0.785398 effort=100 velocity=100
- added joint index_tip: type revolute, parent index_mlp_1, child index_tip_1, origin xyz=-0.001368 0.002219 0.029887 rpy=0 0 0, axis 0.087977 0.993678 -0.069746, limit lower=0.0 upper=0.785398 effort=100 velocity=100
- added joint index_yaw: type revolute, parent index_bulk_1, child index_knuckle_1, origin xyz=-0.003905 0.009839 0.084891 rpy=0 0 0, axis -0.99606 0.086969 -0.017358, limit lower=-0.349066 upper=0.349066 effort=100 velocity=100
- added joint middle_bulk: type fixed, parent index_bulk_1, child middle_bulk_1, origin xyz=0.0 0.006 0.0 rpy=0 0 0
- added joint middle_knuckle: type revolute, parent middle_plp_1, child middle_mlp_1, origin xyz=-0.004 -0.002 0.04725 rpy=0 0 0, axis 0.0 1.0 0.0, limit lower=0.0 upper=0.785398 effort=100 velocity=100
- added joint middle_pitch: type revolute, parent middle_knuckle_1, child middle_plp_1, origin xyz=0.00775 0.008 0.004 rpy=0 0 0, axis 0.0 1.0 0.0, limit lower=0.0 upper=0.785398 effort=100 velocity=100
- added joint middle_tip: type revolute, parent middle_mlp_1, child middle_tip_1, origin xyz=0.0 0.0 0.0315 rpy=0 0 0, axis 0.0 1.0 0.0, limit lower=0.0 upper=0.785398 effort=100 velocity=100
- added joint middle_yaw: type revolute, parent middle_bulk_1, child middle_knuckle_1, origin xyz=-0.002866 -0.02 0.091 rpy=0 0 0, axis -1.0 0.0 0.0, limit lower=-0.349066 upper=0.349066 effort=100 velocity=100
- added joint pinky_knuckle: type revolute, parent pinky_plp_1, child pinky_mlp_1, origin xyz=-0.002512 -0.010584 0.039323 rpy=0 0 0, axis -0.194878 0.965338 0.173624, limit lower=0.0 upper=0.785398 effort=100 velocity=100
- added joint pinky_pitch: type revolute, parent pinky_knuckle_1, child pinky_plp_1, origin xyz=0.006112 0.008539 0.005458 rpy=0 0 0, axis -0.194878 0.965338 0.173624, limit lower=0.0 upper=0.785398 effort=100 velocity=100
- added joint pinky_tip: type revolute, parent pinky_mlp_1, child pinky_tip_1, origin xyz=0.000475 -0.004685 0.026586 rpy=0 0 0, axis -0.194878 0.965338 0.173624, limit lower=0.0 upper=0.785398 effort=100 velocity=100
- added joint pinky_yaw: type revolute, parent pinky_bulk_1, child pinky_knuckle_1, origin xyz=-0.001436 -0.030245 0.078763 rpy=0 0 0, axis -0.98067 -0.194947 -0.016825, limit lower=-0.349066 upper=0.349066 effort=100 velocity=100
- added joint ring_bulk: type fixed, parent middle_bulk_1, child ring_bulk_1, origin xyz=0.0 -0.029 0.0 rpy=0 0 0
- added joint ring_knuckle: type revolute, parent ring_plp_1, child ring_mlp_1, origin xyz=-0.003379 -0.007829 0.044426 rpy=0 0 0, axis -0.086225 0.989495 0.116038, limit lower=0.0 upper=0.785398 effort=100 velocity=100
- added joint ring_pitch: type revolute, parent ring_knuckle_1, child ring_plp_1, origin xyz=0.007067 0.008125 0.004909 rpy=0 0 0, axis -0.086225 0.989495 0.116038, limit lower=0.0 upper=0.785398 effort=100 velocity=100
- added joint ring_tip: type revolute, parent ring_mlp_1, child ring_tip_1, origin xyz=0.000272 -0.003471 0.029797 rpy=0 0 0, axis -0.086225 0.989495 0.116038, limit lower=0.0 upper=0.785398 effort=100 velocity=100
- added joint ring_yaw: type revolute, parent ring_bulk_1, child ring_knuckle_1, origin xyz=-0.002001 -0.015638 0.087079 rpy=0 0 0, axis -0.996234 -0.086694 -0.001008, limit lower=-0.349066 upper=0.349066 effort=100 velocity=100
- added joint thumb_knuckle: type revolute, parent thumb_plp_1, child thumb_mlp_1, origin xyz=0.020792 0.040256 0.039602 rpy=0 0 0, axis 0.864969 -0.501821 -0.002105, limit lower=0.0 upper=0.785398 effort=100 velocity=100
- added joint thumb_pitch: type revolute, parent thumb_cmc_a_1, child thumb_plp_1, origin xyz=0.010924 0.002655 0.007762 rpy=0 0 0, axis 0.864969 -0.501821 -0.002105, limit lower=0.0 upper=1.047198 effort=100 velocity=100
- added joint thumb_roll: type revolute, parent thumb_cmc_b_1, child thumb_cmc_a_1, origin xyz=0.002822 0.004903 -0.009193 rpy=0 0 0, axis -0.35613 -0.610881 -0.707104, limit lower=0.0 upper=0.349066 effort=100 velocity=100
- added joint thumb_tip: type revolute, parent thumb_mlp_1, child thumb_tip_1, origin xyz=0.014837 0.025461 0.027049 rpy=0 0 0, axis 0.864969 -0.501821 -0.002105, limit lower=0.0 upper=0.785398 effort=100 velocity=100
- added joint thumb_yaw: type revolute, parent middle_bulk_1, child thumb_cmc_b_1, origin xyz=0.026917 -0.00751 0.012735 rpy=0 0 0, axis 0.353553 0.612372 -0.707107, limit lower=0.0 upper=0.872665 effort=100 velocity=100
- added joint wrist_pitch_lower: type revolute, parent forearm_1, child wrist_lower_1, origin xyz=-0.012 -0.0217 0.203 rpy=0 0 0, axis 0.0 -1.0 0.0, limit lower=-0.523599 upper=0.523599 effort=100 velocity=100
- added joint wrist_pitch_upper: type revolute, parent wrist_upper_1, child index_bulk_1, origin xyz=0.012 0.021 0.023266 rpy=0 0 0, axis -0.0 -1.0 -0.0, limit lower=-0.349066 upper=0.349066 effort=100 velocity=100
- joint wrist_yaw: child wrist-upper_1 -> wrist_upper_1; parent wrist-lower_1 -> wrist_lower_1
