Commit message: Added additional upper wrist joint

File: urdf/dexhand.xacro (robot description, xacro)
@@ -86,5 +86,5 @@
 <link name="index_bulk_1">
   <inertial>
-    <origin xyz="0.001953836875769263 0.005732502869548333 0.04310739786858114" rpy="0 0 0"/>
+    <origin xyz="0.0019538368757692874 0.005732502869548347 0.0431073978685812" rpy="0 0 0"/>
     <mass value="0.10571474174321724"/>
     <inertia ixx="0.000112" iyy="0.000114" izz="8e-06" ixy="-0.0" iyz="-6e-06" ixz="-7e-06"/>
@@ -106,6 +106,6 @@
 <link name="middle_bulk_1">
   <inertial>
-    <origin xyz="0.01064695002640492 -0.0158135798135519 0.030689623412746947" rpy="0 0 0"/>
-    <mass value="0.23199631248210004"/>
+    <origin xyz="0.010646950026404926 -0.0158135798135519 0.030689623412747002" rpy="0 0 0"/>
+    <mass value="0.2319963124821001"/>
     <inertia ixx="0.000258" iyy="0.000268" izz="7.1e-05" ixy="-1.4e-05" iyz="4.2e-05" ixz="4e-05"/>
   </inertial>
@@ -126,5 +126,5 @@
 <link name="ring_bulk_1">
   <inertial>
-    <origin xyz="0.003391811603104285 -0.01025124324374128 0.05277806405684754" rpy="0 0 0"/>
+    <origin xyz="0.003391811603104299 -0.010251243243741267 0.052778064056847374" rpy="0 0 0"/>
     <mass value="0.09588694429304498"/>
     <inertia ixx="7.4e-05" iyy="7.4e-05" izz="7e-06" ixy="1e-06" iyz="8e-06" ixz="-7e-06"/>
@@ -146,5 +146,5 @@
 <link name="index_knuckle_1">
   <inertial>
-    <origin xyz="0.007134673083101478 -0.0005540875413111747 0.0011013348331220807" rpy="0 0 0"/>
+    <origin xyz="0.007134673083101494 -0.000554087541311192 0.0011013348331223027" rpy="0 0 0"/>
     <mass value="0.016772407452453803"/>
     <inertia ixx="1e-06" iyy="1e-06" izz="1e-06" ixy="0.0" iyz="0.0" ixz="-0.0"/>
@@ -166,5 +166,5 @@
 <link name="middle_knuckle_1">
   <inertial>
-    <origin xyz="0.006935399474227782 3.095281810635425e-08 0.0009794888636300847" rpy="0 0 0"/>
+    <origin xyz="0.006935399474227786 3.095281810115008e-08 0.0009794888636301402" rpy="0 0 0"/>
     <mass value="0.016772407452453803"/>
     <inertia ixx="1e-06" iyy="1e-06" izz="1e-06" ixy="0.0" iyz="0.0" ixz="-0.0"/>
@@ -186,5 +186,5 @@
 <link name="ring_knuckle_1">
   <inertial>
-    <origin xyz="0.006918049206992894 0.0004875294278836907 0.0009797412002323647" rpy="0 0 0"/>
+    <origin xyz="0.006918049206992899 0.000487529427883715 0.0009797412002321981" rpy="0 0 0"/>
     <mass value="0.016772407452453803"/>
     <inertia ixx="1e-06" iyy="1e-06" izz="1e-06" ixy="-0.0" iyz="-0.0" ixz="-0.0"/>
@@ -206,10 +206,10 @@
 <link name="pinky_knuckle_1">
   <inertial>
-    <origin xyz="0.006818820473942549 0.0011824337110899266 0.0010801856787569508" rpy="0 0 0"/>
+    <origin xyz="0.006818820473942532 0.0011821873591725332 0.0010801856787559516" rpy="0 0 0"/>
     <mass value="0.016772407452453803"/>
     <inertia ixx="1e-06" iyy="1e-06" izz="1e-06" ixy="-0.0" iyz="-0.0" ixz="-0.0"/>
   </inertial>
   <visual>
-    <origin xyz="0.013416 0.038945 -0.334029" rpy="0 0 0"/>
+    <origin xyz="0.013416 0.038988 -0.334029" rpy="0 0 0"/>
     <geometry>
       <mesh filename="package://dexhand_description/meshes/pinky_knuckle_1.stl" scale="0.001 0.001 0.001"/>
@@ -218,5 +218,5 @@
   </visual>
   <collision>
-    <origin xyz="0.013416 0.038945 -0.334029" rpy="0 0 0"/>
+    <origin xyz="0.013416 0.038988 -0.334029" rpy="0 0 0"/>
     <geometry>
       <mesh filename="package://dexhand_description/meshes/pinky_knuckle_1.stl" scale="0.001 0.001 0.001"/>
@@ -226,5 +226,5 @@
 <link name="index_plp_1">
   <inertial>
-    <origin xyz="-0.006869198158126709 -0.006033909809302199 0.022940465298997237" rpy="0 0 0"/>
+    <origin xyz="-0.006869198158126683 -0.006033909809302226 0.022940465298997237" rpy="0 0 0"/>
     <mass value="0.051567105457974535"/>
     <inertia ixx="1.1e-05" iyy="1.1e-05" izz="2e-06" ixy="-0.0" iyz="-1e-06" ixz="0.0"/>
@@ -246,5 +246,5 @@
 <link name="index_mlp_1">
   <inertial>
-    <origin xyz="-0.0014672452336520862 -0.004861924263139264 0.014904028884496323" rpy="0 0 0"/>
+    <origin xyz="-0.0014672452336520724 -0.004861924263139264 0.014904028884496767" rpy="0 0 0"/>
     <mass value="0.017288956361389173"/>
     <inertia ixx="1e-06" iyy="1e-06" izz="0.0" ixy="-0.0" iyz="-0.0" ixz="-0.0"/>
@@ -266,5 +266,5 @@
 <link name="index_tip_1">
   <inertial>
-    <origin xyz="-0.000864193964734649 -0.005385771025884167 0.006769569897979166" rpy="0 0 0"/>
+    <origin xyz="-0.0008641939647346161 -0.005385771025884202 0.006769569897979" rpy="0 0 0"/>
     <mass value="0.0160783570939756"/>
     <inertia ixx="1e-06" iyy="1e-06" izz="0.0" ixy="-0.0" iyz="-0.0" ixz="0.0"/>
@@ -284,12 +284,292 @@
   </collision>
 </link>
+<link name="middle_plp_1">
+  <inertial>
+    <origin xyz="-0.00594358104054421 -0.00819999164061916 0.02373210744114279" rpy="0 0 0"/>
+    <mass value="0.05600912510930776"/>
+    <inertia ixx="1.3e-05" iyy="1.3e-05" izz="2e-06" ixy="0.0" iyz="0.0" ixz="0.0"/>
+  </inertial>
+  <visual>
+    <origin xyz="0.007096 -0.0143 -0.350266" rpy="0 0 0"/>
+    <geometry>
+      <mesh filename="package://dexhand_description/meshes/middle_plp_1.stl" scale="0.001 0.001 0.001"/>
+    </geometry>
+    <material name="silver"/>
+  </visual>
+  <collision>
+    <origin xyz="0.007096 -0.0143 -0.350266" rpy="0 0 0"/>
+    <geometry>
+      <mesh filename="package://dexhand_description/meshes/middle_plp_1.stl" scale="0.001 0.001 0.001"/>
+    </geometry>
+  </collision>
+</link>
+<link name="middle_mlp_1">
+  <inertial>
+    <origin xyz="-0.0002942937668230401 -0.006300032078833909 0.01528820861860336" rpy="0 0 0"/>
+    <mass value="0.019660714741942815"/>
+    <inertia ixx="1e-06" iyy="1e-06" izz="1e-06" ixy="0.0" iyz="0.0" ixz="-0.0"/>
+  </inertial>
+  <visual>
+    <origin xyz="0.011096 -0.0123 -0.397516" rpy="0 0 0"/>
+    <geometry>
+      <mesh filename="package://dexhand_description/meshes/middle_mlp_1.stl" scale="0.001 0.001 0.001"/>
+    </geometry>
+    <material name="silver"/>
+  </visual>
+  <collision>
+    <origin xyz="0.011096 -0.0123 -0.397516" rpy="0 0 0"/>
+    <geometry>
+      <mesh filename="package://dexhand_description/meshes/middle_mlp_1.stl" scale="0.001 0.001 0.001"/>
+    </geometry>
+  </collision>
+</link>
+<link name="middle_tip_1">
+  <inertial>
+    <origin xyz="-0.0006361624064090965 -0.006200060330852975 0.0068547001404333785" rpy="0 0 0"/>
+    <mass value="0.0177222165691614"/>
+    <inertia ixx="1e-06" iyy="1e-06" izz="0.0" ixy="0.0" iyz="0.0" ixz="0.0"/>
+  </inertial>
+  <visual>
+    <origin xyz="0.011096 -0.0123 -0.429016" rpy="0 0 0"/>
+    <geometry>
+      <mesh filename="package://dexhand_description/meshes/middle_tip_1.stl" scale="0.001 0.001 0.001"/>
+    </geometry>
+    <material name="silver"/>
+  </visual>
+  <collision>
+    <origin xyz="0.011096 -0.0123 -0.429016" rpy="0 0 0"/>
+    <geometry>
+      <mesh filename="package://dexhand_description/meshes/middle_tip_1.stl" scale="0.001 0.001 0.001"/>
+    </geometry>
+  </collision>
+</link>
+<link name="ring_plp_1">
+  <inertial>
+    <origin xyz="-0.004988778025381051 -0.011235452676283293 0.021431089299078443" rpy="0 0 0"/>
+    <mass value="0.051607390430851795"/>
+    <inertia ixx="1.1e-05" iyy="1.1e-05" izz="2e-06" ixy="0.0" iyz="1e-06" ixz="-0.0"/>
+  </inertial>
+  <visual>
+    <origin xyz="0.006914 0.010213 -0.347254" rpy="0 0 0"/>
+    <geometry>
+      <mesh filename="package://dexhand_description/meshes/ring_plp_1.stl" scale="0.001 0.001 0.001"/>
+    </geometry>
+    <material name="silver"/>
+  </visual>
+  <collision>
+    <origin xyz="0.006914 0.010213 -0.347254" rpy="0 0 0"/>
+    <geometry>
+      <mesh filename="package://dexhand_description/meshes/ring_plp_1.stl" scale="0.001 0.001 0.001"/>
+    </geometry>
+  </collision>
+</link>
+<link name="ring_mlp_1">
+  <inertial>
+    <origin xyz="0.00037321408367821905 -0.007644713369413636 0.013759338633879237" rpy="0 0 0"/>
+    <mass value="0.017289443732746056"/>
+    <inertia ixx="1e-06" iyy="1e-06" izz="0.0" ixy="0.0" iyz="0.0" ixz="-0.0"/>
+  </inertial>
+  <visual>
+    <origin xyz="0.010293 0.018042 -0.39168" rpy="0 0 0"/>
+    <geometry>
+      <mesh filename="package://dexhand_description/meshes/ring_mlp_1.stl" scale="0.001 0.001 0.001"/>
+    </geometry>
+    <material name="silver"/>
+  </visual>
+  <collision>
+    <origin xyz="0.010293 0.018042 -0.39168" rpy="0 0 0"/>
+    <geometry>
+      <mesh filename="package://dexhand_description/meshes/ring_mlp_1.stl" scale="0.001 0.001 0.001"/>
+    </geometry>
+  </collision>
+</link>
+<link name="ring_tip_1">
+  <inertial>
+    <origin xyz="-2.475222624376619e-05 -0.006623152446546359 0.005616048262013451" rpy="0 0 0"/>
+    <mass value="0.016038982608931798"/>
+    <inertia ixx="1e-06" iyy="1e-06" izz="0.0" ixy="0.0" iyz="0.0" ixz="0.0"/>
+  </inertial>
+  <visual>
+    <origin xyz="0.010021 0.021513 -0.421477" rpy="0 0 0"/>
+    <geometry>
+      <mesh filename="package://dexhand_description/meshes/ring_tip_1.stl" scale="0.001 0.001 0.001"/>
+    </geometry>
+    <material name="silver"/>
+  </visual>
+  <collision>
+    <origin xyz="0.010021 0.021513 -0.421477" rpy="0 0 0"/>
+    <geometry>
+      <mesh filename="package://dexhand_description/meshes/ring_tip_1.stl" scale="0.001 0.001 0.001"/>
+    </geometry>
+  </collision>
+</link>
+<link name="pinky_plp_1">
+  <inertial>
+    <origin xyz="-0.0038106689386204866 -0.012544392770237969 0.01824146705848928" rpy="0 0 0"/>
+    <mass value="0.04272741599660885"/>
+    <inertia ixx="8e-06" iyy="8e-06" izz="1e-06" ixy="0.0" iyz="1e-06" ixz="-0.0"/>
+  </inertial>
+  <visual>
+    <origin xyz="0.007304 0.030449 -0.339487" rpy="0 0 0"/>
+    <geometry>
+      <mesh filename="package://dexhand_description/meshes/pinky_plp_1.stl" scale="0.001 0.001 0.001"/>
+    </geometry>
+    <material name="silver"/>
+  </visual>
+  <collision>
+    <origin xyz="0.007304 0.030449 -0.339487" rpy="0 0 0"/>
+    <geometry>
+      <mesh filename="package://dexhand_description/meshes/pinky_plp_1.stl" scale="0.001 0.001 0.001"/>
+    </geometry>
+  </collision>
+</link>
+<link name="pinky_mlp_1">
+  <inertial>
+    <origin xyz="0.0010481249693847592 -0.007529779935539188 0.011942260100063107" rpy="0 0 0"/>
+    <mass value="0.012979924052628225"/>
+    <inertia ixx="1e-06" iyy="1e-06" izz="0.0" ixy="0.0" iyz="0.0" ixz="-0.0"/>
+  </inertial>
+  <visual>
+    <origin xyz="0.009816 0.041033 -0.37881" rpy="0 0 0"/>
+    <geometry>
+      <mesh filename="package://dexhand_description/meshes/pinky_mlp_1.stl" scale="0.001 0.001 0.001"/>
+    </geometry>
+    <material name="silver"/>
+  </visual>
+  <collision>
+    <origin xyz="0.009816 0.041033 -0.37881" rpy="0 0 0"/>
+    <geometry>
+      <mesh filename="package://dexhand_description/meshes/pinky_mlp_1.stl" scale="0.001 0.001 0.001"/>
+    </geometry>
+  </collision>
+</link>
+<link name="pinky_tip_1">
+  <inertial>
+    <origin xyz="0.0005692184398215679 -0.006140507616860642 0.004252021497513858" rpy="0 0 0"/>
+    <mass value="0.012880734939160096"/>
+    <inertia ixx="1e-06" iyy="1e-06" izz="0.0" ixy="0.0" iyz="0.0" ixz="0.0"/>
+  </inertial>
+  <visual>
+    <origin xyz="0.009341 0.045718 -0.405396" rpy="0 0 0"/>
+    <geometry>
+      <mesh filename="package://dexhand_description/meshes/pinky_tip_1.stl" scale="0.001 0.001 0.001"/>
+    </geometry>
+    <material name="silver"/>
+  </visual>
+  <collision>
+    <origin xyz="0.009341 0.045718 -0.405396" rpy="0 0 0"/>
+    <geometry>
+      <mesh filename="package://dexhand_description/meshes/pinky_tip_1.stl" scale="0.001 0.001 0.001"/>
+    </geometry>
+  </collision>
+</link>
+<link name="thumb_cmc_b_1">
+  <inertial>
+    <origin xyz="0.0033512527298519643 0.005810607163787045 -0.008141548652481512" rpy="0 0 0"/>
+    <mass value="0.008494087027059793"/>
+    <inertia ixx="0.0" iyy="0.0" izz="0.0" ixy="-0.0" iyz="0.0" ixz="0.0"/>
+  </inertial>
+  <visual>
+    <origin xyz="-0.014937 -0.01879 -0.268001" rpy="0 0 0"/>
+    <geometry>
+      <mesh filename="package://dexhand_description/meshes/thumb_cmc_b_1.stl" scale="0.001 0.001 0.001"/>
+    </geometry>
+    <material name="silver"/>
+  </visual>
+  <collision>
+    <origin xyz="-0.014937 -0.01879 -0.268001" rpy="0 0 0"/>
+    <geometry>
+      <mesh filename="package://dexhand_description/meshes/thumb_cmc_b_1.stl" scale="0.001 0.001 0.001"/>
+    </geometry>
+  </collision>
+</link>
+<link name="thumb_cmc_a_1">
+  <inertial>
+    <origin xyz="0.0029466810384300712 0.005054293341482698 0.005851296597689126" rpy="0 0 0"/>
+    <mass value="0.015039242610946097"/>
+    <inertia ixx="0.0" iyy="0.0" izz="0.0" ixy="0.0" iyz="-0.0" ixz="-0.0"/>
+  </inertial>
+  <visual>
+    <origin xyz="-0.017759 -0.023693 -0.258808" rpy="0 0 0"/>
+    <geometry>
+      <mesh filename="package://dexhand_description/meshes/thumb_cmc_a_1.stl" scale="0.001 0.001 0.001"/>
+    </geometry>
+    <material name="silver"/>
+  </visual>
+  <collision>
+    <origin xyz="-0.017759 -0.023693 -0.258808" rpy="0 0 0"/>
+    <geometry>
+      <mesh filename="package://dexhand_description/meshes/thumb_cmc_a_1.stl" scale="0.001 0.001 0.001"/>
+    </geometry>
+  </collision>
+</link>
+<link name="thumb_plp_1">
+  <inertial>
+    <origin xyz="0.005433746290735154 0.025637034957291558 0.01661470656693176" rpy="0 0 0"/>
+    <mass value="0.06710748615776632"/>
+    <inertia ixx="2e-05" iyy="1.5e-05" izz="1.3e-05" ixy="-5e-06" iyz="-9e-06" ixz="-5e-06"/>
+  </inertial>
+  <visual>
+    <origin xyz="-0.028683 -0.026348 -0.26657" rpy="0 0 0"/>
+    <geometry>
+      <mesh filename="package://dexhand_description/meshes/thumb_plp_1.stl" scale="0.001 0.001 0.001"/>
+    </geometry>
+    <material name="silver"/>
+  </visual>
+  <collision>
+    <origin xyz="-0.028683 -0.026348 -0.26657" rpy="0 0 0"/>
+    <geometry>
+      <mesh filename="package://dexhand_description/meshes/thumb_plp_1.stl" scale="0.001 0.001 0.001"/>
+    </geometry>
+  </collision>
+</link>
+<link name="thumb_mlp_1">
+  <inertial>
+    <origin xyz="0.002151568364903468 0.015611380274394432 0.012743956202626694" rpy="0 0 0"/>
+    <mass value="0.025187203449803457"/>
+    <inertia ixx="2e-06" iyy="2e-06" izz="2e-06" ixy="-0.0" iyz="-1e-06" ixz="-0.0"/>
+  </inertial>
+  <visual>
+    <origin xyz="-0.049475 -0.066604 -0.306172" rpy="0 0 0"/>
+    <geometry>
+      <mesh filename="package://dexhand_description/meshes/thumb_mlp_1.stl" scale="0.001 0.001 0.001"/>
+    </geometry>
+    <material name="silver"/>
+  </visual>
+  <collision>
+    <origin xyz="-0.049475 -0.066604 -0.306172" rpy="0 0 0"/>
+    <geometry>
+      <mesh filename="package://dexhand_description/meshes/thumb_mlp_1.stl" scale="0.001 0.001 0.001"/>
+    </geometry>
+  </collision>
+</link>
+<link name="thumb_tip_1">
+  <inertial>
+    <origin xyz="-0.0009246362325293633 0.010131321702323517 0.007474037055237359" rpy="0 0 0"/>
+    <mass value="0.02316990761545859"/>
+    <inertia ixx="2e-06" iyy="2e-06" izz="2e-06" ixy="-0.0" iyz="-1e-06" ixz="-0.0"/>
+  </inertial>
+  <visual>
+    <origin xyz="-0.064312 -0.092065 -0.333221" rpy="0 0 0"/>
+    <geometry>
+      <mesh filename="package://dexhand_description/meshes/thumb_tip_1.stl" scale="0.001 0.001 0.001"/>
+    </geometry>
+    <material name="silver"/>
+  </visual>
+  <collision>
+    <origin xyz="-0.064312 -0.092065 -0.333221" rpy="0 0 0"/>
+    <geometry>
+      <mesh filename="package://dexhand_description/meshes/thumb_tip_1.stl" scale="0.001 0.001 0.001"/>
+    </geometry>
+  </collision>
+</link>
 <link name="pinky_bulk_1">
   <inertial>
-    <origin xyz="0.0027271468848747375 -0.00919661076399992 0.036410887836454076" rpy="0 0 0"/>
+    <origin xyz="0.0027271468848747184 -0.022196857115917325 0.03641088783645313" rpy="0 0 0"/>
     <mass value="0.11417768838788588"/>
     <inertia ixx="0.000111" iyy="0.000112" izz="1e-05" ixy="1e-06" iyz="1.3e-05" ixz="-1e-05"/>
   </inertial>
   <visual>
-    <origin xyz="0.01198 0.0217 -0.255266" rpy="0 0 0"/>
+    <origin xyz="0.01198 0.008743 -0.255266" rpy="0 0 0"/>
     <geometry>
       <mesh filename="package://dexhand_description/meshes/pinky_bulk_1.stl" scale="0.001 0.001 0.001"/>
@@ -298,287 +578,7 @@
   </visual>
   <collision>
-    <origin xyz="0.01198 0.0217 -0.255266" rpy="0 0 0"/>
+    <origin xyz="0.01198 0.008743 -0.255266" rpy="0 0 0"/>
     <geometry>
       <mesh filename="package://dexhand_description/meshes/pinky_bulk_1.stl" scale="0.001 0.001 0.001"/>
-    </geometry>
-  </collision>
-</link>
-<link name="middle_plp_1">
-  <inertial>
-    <origin xyz="-0.005943581040544219 -0.008199991640619155 0.023732107441142736" rpy="0 0 0"/>
-    <mass value="0.05600912510930776"/>
-    <inertia ixx="1.3e-05" iyy="1.3e-05" izz="2e-06" ixy="0.0" iyz="0.0" ixz="0.0"/>
-  </inertial>
-  <visual>
-    <origin xyz="0.007096 -0.0143 -0.350266" rpy="0 0 0"/>
-    <geometry>
-      <mesh filename="package://dexhand_description/meshes/middle_plp_1.stl" scale="0.001 0.001 0.001"/>
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